File: v0.4/THT/Latest/inputs.sch (KiCad schematic (older format))
At the start: 41 parts, among them IC3 Trig Cond Socket, U1 SP721, U3 SP721, U5 MPX4250

Commit message: Folder cleanup
Parts:
- U5: symbol v0.4.4c-rescue:MPX4250-Misc -> v0.4.3d-rescue:MPX4250-Misc-v0.4.4c-rescue
Changed lines of the file:
@@
 $EndDescr
 $Comp
-L v0.4.4c-rescue:MPX4250-Misc U?
+L v0.4.3d-rescue:MPX4250-Misc-v0.4.4c-rescue U?
 U 1 1 5CD196C6
 P 2000 1900
