File: v0.4/THT/Latest/v0.4.3d.sch (KiCad schematic (older format))
At the start: 1 part

Commit message: Folder cleanup
Parts:
- XA1: symbol v0.4.4c-rescue:Arduino_Mega2560_Shield-Arduino -> v0.4.3d-rescue:Arduino_Mega2560_Shield-Arduino-v0.4.4c-rescue
Changed lines of the file:
@@
 $EndDescr
 $Comp
-L v0.4.4c-rescue:Arduino_Mega2560_Shield-Arduino XA1
+L v0.4.3d-rescue:Arduino_Mega2560_Shield-Arduino-v0.4.4c-rescue XA1
 U 1 1 5CD14B53
 P 6050 3400
