File: v0.4/SMD/Latest/inputs.sch (KiCad schematic (older format))
At the start: 44 parts, among them IC3 Trig Cond Socket, U5 MPX4250, U6 SP720

Commit message: Add v0.4.4d SMD design files
Parts:
- U5: symbol Misc:MPX4250 -> v0.4.4c-rescue:MPX4250-Misc
- U6: symbol IC_Automotive:SP720 -> v0.4.4c-rescue:SP720-IC_Automotive
Changed lines of the file:
@@
 EESchema Schematic File Version 4
-LIBS:v0.4.4c-cache
+LIBS:v0.4.4d-cache
 EELAYER 30 0
 EELAYER END
@@
 encoding utf-8
 Sheet 3 7
-Title ""
-Date ""
-Rev ""
-Comp ""
+Title "0.4"
+Date "2021-03-27"
+Rev "4d"
+Comp "Speeduino"
 Comment1 ""
 Comment2 ""
@@
 $EndDescr
 $Comp
-L Misc:MPX4250 U?
+L v0.4.4c-rescue:MPX4250-Misc U?
 U 1 1 5CD196C6
 P 2000 1900
@@
 MAP Sensor
 $Comp
-L IC_Automotive:SP720 U6
+L v0.4.4c-rescue:SP720-IC_Automotive U6
 U 1 1 5CDA8540
 P 8900 1450
