File: v0.4/SMD/Latest/outputs.sch (KiCad schematic (older format))
At the start: 22 parts, among them J2 Conn_01x06, Q1 SSM3K357R, Q2 SSM3K357R, Q3 SSM3K357R, U7 VNLD5090, U9 VNLD5090

Commit message: Add v0.4.4d SMD design files
Parts:
- D16, D17, D18, D19: footprint Diode_SMD:D_SOD-323 -> Diode_SMD:D_SOD-123F; Digikey Part Number 1N4448WXTPMSCT-ND -> S110FACT-ND; Manufacturer_Name MCC -> ONSEMI; Manufacturer_Part_Number 1N4448WX-TP -> S110FA; URL https://www.digikey.com/product-detail/en/micro-commercial-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 -> https://www.digikey.com/en/products/detail/on-semiconductor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
- U7, U9: symbol IC_Automotive:VNLD5090 -> v0.4.4c-rescue:VNLD5090-IC_Automotive
Changed lines of the file:
@@
 EESchema Schematic File Version 4
-LIBS:v0.4.4c-cache
+LIBS:v0.4.4d-cache
 EELAYER 30 0
 EELAYER END
@@
 encoding utf-8
 Sheet 6 7
-Title ""
-Date ""
-Rev ""
-Comp ""
+Title "0.4"
+Date "2021-03-27"
+Rev "4d"
+Comp "Speeduino"
 Comment1 ""
 Comment2 ""
@@
 $EndDescr
 $Comp
-L IC_Automotive:VNLD5090 U7
+L v0.4.4c-rescue:VNLD5090-IC_Automotive U7
 U 1 1 5CE9F50F
 P 2600 1900
@@
 PWM Idle and Boost outputs
 $Comp
-L IC_Automotive:VNLD5090 U9
+L v0.4.4c-rescue:VNLD5090-IC_Automotive U9
 U 1 1 5CEAD71A
 P 8350 1900
@@
 Text Notes 4750 3300 0    78   ~ 0
 Fan and Fuel Pump outputs
-$Comp
-L Device:D D18
-U 1 1 5CEC935F
-P 3850 2300
-F 0 "D18" V 3896 2221 50  0000 R CNN
-F 1 "D" V 3805 2221 50  0000 R CNN
-F 2 "Diode_SMD:D_SOD-323" H 3850 2300 50  0001 C CNN
-F 3 "~" H 3850 2300 50  0001 C CNN
-F 4 "1N4448WXTPMSCT-ND" H 0   0   50  0001 C CNN "Digikey Part Number"
-F 5 "MCC" H 0   0   50  0001 C CNN "Manufacturer_Name"
-F 6 "1N4448WX-TP" H 0   0   50  0001 C CNN "Manufacturer_Part_Number"
-F 7 "https://www.digikey.com/product-detail/en/micro-commercial-co/1N4448WX-TP/1N4448WXTPMSCT-ND/789338" H 0   0   50  0001 C CNN "URL"
-	1    3850 2300
-	0    -1   -1   0
-$EndComp
-$Comp
-L Device:D D17
-U 1 1 5CEC9E8B
-P 3850 1400
-F 0 "D17" V 3804 1479 50  0000 L CNN
-F 1 "D" V 3895 1479 50  0000 L CNN
-F 2 "Diode_SMD:D_SOD-323" H 3850 1400 50  0001 C CNN
-F 3 "~" H 3850 1400 50  0001 C CNN
-F 4 "1N4448WXTPMSCT-ND" H 0   0   50  0001 C CNN "Digikey Part Number"
-F 5 "MCC" H 0   0   50  0001 C CNN "Manufacturer_Name"
-F 6 "1N4448WX-TP" H 0   0   50  0001 C CNN "Manufacturer_Part_Number"
-F 7 "https://www.digikey.com/product-detail/en/micro-commercial-co/1N4448WX-TP/1N4448WXTPMSCT-ND/789338" H 0   0   50  0001 C CNN "URL"
-	1    3850 1400
-	0    1    1    0
-$EndComp
 Text GLabel 3700 2500 0    50   Input ~ 0
 12V-SW
@@
 F 0 "D19" V 9304 1579 50  0000 L CNN
 F 1 "D" V 9395 1579 50  0000 L CNN
-F 2 "Diode_SMD:D_SOD-323" H 9350 1500 50  0001 C CNN
+F 2 "Diode_SMD:D_SOD-123F" H 9350 1500 50  0001 C CNN
 F 3 "~" H 9350 1500 50  0001 C CNN
-F 4 "1N4448WXTPMSCT-ND" H 0   0   50  0001 C CNN "Digikey Part Number"
-F 5 "MCC" H 0   0   50  0001 C CNN "Manufacturer_Name"
-F 6 "1N4448WX-TP" H 0   0   50  0001 C CNN "Manufacturer_Part_Number"
-F 7 "https://www.digikey.com/product-detail/en/micro-commercial-co/1N4448WX-TP/1N4448WXTPMSCT-ND/789338" H 0   0   50  0001 C CNN "URL"
+F 4 "S110FACT-ND" H 0   0   50  0001 C CNN "Digikey Part Number"
+F 5 "ONSEMI" H 0   0   50  0001 C CNN "Manufacturer_Name"
+F 6 "S110FA" H 0   0   50  0001 C CNN "Manufacturer_Part_Number"
+F 7 "https://www.digikey.com/en/products/detail/on-semiconductor/S110FA/5892098" H 0   0   50  0001 C CNN "URL"
 	1    9350 1500
 	0    1    1    0
@@
 Text GLabel 7150 2000 0    50   Input ~ 0
 MCU-D4
-$Comp
-L Device:D D16
-U 1 1 5D1AF048
-P 9350 2350
-F 0 "D16" V 9304 2429 50  0000 L CNN
-F 1 "D" V 9395 2429 50  0000 L CNN
-F 2 "Diode_SMD:D_SOD-323" H 9350 2350 50  0001 C CNN
-F 3 "~" H 9350 2350 50  0001 C CNN
-F 4 "1N4448WXTPMSCT-ND" H 0   0   50  0001 C CNN "Digikey Part Number"
-F 5 "MCC" H 0   0   50  0001 C CNN "Manufacturer_Name"
-F 6 "1N4448WX-TP" H 0   0   50  0001 C CNN "Manufacturer_Part_Number"
-F 7 "https://www.digikey.com/product-detail/en/micro-commercial-co/1N4448WX-TP/1N4448WXTPMSCT-ND/789338" H 0   0   50  0001 C CNN "URL"
-	1    9350 2350
-	0    1    -1   0
-$EndComp
 Text GLabel 9550 2600 2    50   Input ~ 0
 12V-SW
@@
 	0    1    1    0
 $EndComp
+$Comp
+L Device:D D16
+U 1 1 605C7132
+P 9350 2350
+F 0 "D16" V 9304 2429 50  0000 L CNN
+F 1 "D" V 9395 2429 50  0000 L CNN
+F 2 "Diode_SMD:D_SOD-123F" H 9350 2350 50  0001 C CNN
+F 3 "~" H 9350 2350 50  0001 C CNN
+F 4 "S110FACT-ND" H 0   850 50  0001 C CNN "Digikey Part Number"
+F 5 "ONSEMI" H 0   850 50  0001 C CNN "Manufacturer_Name"
+F 6 "S110FA" H 0   850 50  0001 C CNN "Manufacturer_Part_Number"
+F 7 "https://www.digikey.com/en/products/detail/on-semiconductor/S110FA/5892098" H 0   850 50  0001 C CNN "URL"
+	1    9350 2350
+	0    1    -1   0
+$EndComp
+$Comp
+L Device:D D17
+U 1 1 605CAD9E
+P 3850 1400
+F 0 "D17" V 3804 1479 50  0000 L CNN
+F 1 "D" V 3895 1479 50  0000 L CNN
+F 2 "Diode_SMD:D_SOD-123F" H 3850 1400 50  0001 C CNN
+F 3 "~" H 3850 1400 50  0001 C CNN
+F 4 "S110FACT-ND" H -5500 -100 50  0001 C CNN "Digikey Part Number"
+F 5 "ONSEMI" H -5500 -100 50  0001 C CNN "Manufacturer_Name"
+F 6 "S110FA" H -5500 -100 50  0001 C CNN "Manufacturer_Part_Number"
+F 7 "https://www.digikey.com/en/products/detail/on-semiconductor/S110FA/5892098" H -5500 -100 50  0001 C CNN "URL"
+	1    3850 1400
+	0    1    1    0
+$EndComp
+$Comp
+L Device:D D18
+U 1 1 605CC406
+P 3850 2300
+F 0 "D18" V 3804 2379 50  0000 L CNN
+F 1 "D" V 3895 2379 50  0000 L CNN
+F 2 "Diode_SMD:D_SOD-123F" H 3850 2300 50  0001 C CNN
+F 3 "~" H 3850 2300 50  0001 C CNN
+F 4 "S110FACT-ND" H -5500 800 50  0001 C CNN "Digikey Part Number"
+F 5 "ONSEMI" H -5500 800 50  0001 C CNN "Manufacturer_Name"
+F 6 "S110FA" H -5500 800 50  0001 C CNN "Manufacturer_Part_Number"
+F 7 "https://www.digikey.com/en/products/detail/on-semiconductor/S110FA/5892098" H -5500 800 50  0001 C CNN "URL"
+	1    3850 2300
+	0    1    -1   0
+$EndComp
 $EndSCHEMATC
