File: PNPs/Miata NA6/Prior versions/v1.2/inputs.sch (KiCad schematic (older format))
At the start: 39 parts, among them U11 KP234, U5 MPX4250, U6 SP720

Commit message: NA6 PNP v1.3 files
Parts:
- removed C29: 0.01uF, Capacitor_SMD:C_0805_2012Metric, symbol Device:C
- removed C30: 1uF, Capacitor_SMD:C_0805_2012Metric, symbol Device:C
- removed C31: 0.1uF, Capacitor_SMD:C_0805_2012Metric, symbol Device:C
- removed R67: 22K, Resistor_SMD:R_0805_2012Metric, symbol Device:R
- removed U11: KP234, Misc:KP234, symbol Misc:KP234
Connections:
- net labels removed: MCU-A12
- wire segments 155 -> 140
Other:
- note removed: "Baro Sensor"
Changed lines of the file:
@@
 Wire Wire Line
 	5900 6300 5900 6450
-$Comp
-L power:GND #PWR0114
-U 1 1 5F6DC469
-P 8450 6250
-F 0 "#PWR0114" H 8450 6000 50  0001 C CNN
-F 1 "GND" V 8455 6122 50  0000 R CNN
-F 2 "" H 8450 6250 50  0001 C CNN
-F 3 "" H 8450 6250 50  0001 C CNN
-	1    8450 6250
-	0    1    1    0
-$EndComp
-$Comp
-L power:GND #PWR0115
-U 1 1 5F6DC46F
-P 9550 5450
-F 0 "#PWR0115" H 9550 5200 50  0001 C CNN
-F 1 "GND" H 9555 5277 50  0000 C CNN
-F 2 "" H 9550 5450 50  0001 C CNN
-F 3 "" H 9550 5450 50  0001 C CNN
-	1    9550 5450
-	-1   0    0    1
-$EndComp
-Wire Wire Line
-	9550 5950 9550 5850
-Wire Wire Line
-	9550 5950 9800 5950
-$Comp
-L power:VDDA #PWR0116
-U 1 1 5F6DC477
-P 8300 5600
-F 0 "#PWR0116" H 8300 5450 50  0001 C CNN
-F 1 "VDDA" V 8318 5728 50  0000 L CNN
-F 2 "" H 8300 5600 50  0001 C CNN
-F 3 "" H 8300 5600 50  0001 C CNN
-	1    8300 5600
-	0    -1   -1   0
-$EndComp
-$Comp
-L Device:C C29
-U 1 1 5F6DC481
-P 8550 5400
-F 0 "C29" H 8350 5450 50  0000 L CNN
-F 1 "0.01uF" H 8250 5350 50  0000 L CNN
-F 2 "Capacitor_SMD:C_0805_2012Metric" H 8588 5250 50  0001 C CNN
-F 3 "~" H 8550 5400 50  0001 C CNN
-F 4 "311-1136-1-ND" H 8550 5400 50  0001 C CNN "Digikey Part Number"
-F 5 "Yageo" H 8550 5400 50  0001 C CNN "Manufacturer_Name"
-F 6 "CC0805KRX7R9BB103" H 8550 5400 50  0001 C CNN "Manufacturer_Part_Number"
-F 7 "https://www.digikey.com/product-detail/en/yageo/CC0805KRX7R9BB103/311-1136-1-ND/303046" H 8550 5400 50  0001 C CNN "URL"
-	1    8550 5400
-	1    0    0    -1
-$EndComp
-$Comp
-L Device:C C30
-U 1 1 5F6DC48B
-P 8850 5400
-F 0 "C30" H 8965 5446 50  0000 L CNN
-F 1 "1uF" H 8965 5355 50  0000 L CNN
-F 2 "Capacitor_SMD:C_0805_2012Metric" H 8888 5250 50  0001 C CNN
-F 3 "~" H 8850 5400 50  0001 C CNN
-F 4 "311-1365-1-ND" H 8850 5400 50  0001 C CNN "Digikey Part Number"
-F 5 "Yageo" H 8850 5400 50  0001 C CNN "Manufacturer_Name"
-F 6 "CC0805KKX7R7BB105" H 8850 5400 50  0001 C CNN "Manufacturer_Part_Number"
-F 7 "https://www.digikey.com/product-detail/en/yageo/CC0805KKX7R7BB105/311-1365-1-ND/2103149" H 8850 5400 50  0001 C CNN "URL"
-	1    8850 5400
-	1    0    0    -1
-$EndComp
-$Comp
-L power:GND #PWR0117
-U 1 1 5F6DC491
-P 8700 5200
-F 0 "#PWR0117" H 8700 4950 50  0001 C CNN
-F 1 "GND" H 8705 5027 50  0000 C CNN
-F 2 "" H 8700 5200 50  0001 C CNN
-F 3 "" H 8700 5200 50  0001 C CNN
-	1    8700 5200
-	-1   0    0    1
-$EndComp
-Text Notes 8650 4900 0    74   ~ 0
-Baro Sensor
-Text GLabel 9800 5950 2    50   Input ~ 0
-MCU-A12
-Wire Wire Line
-	8550 5250 8700 5250
-Wire Wire Line
-	8300 5600 8550 5600
-Wire Wire Line
-	8700 5600 8700 5650
-Wire Wire Line
-	8550 5550 8550 5600
-Connection ~ 8550 5600
-Wire Wire Line
-	8550 5600 8700 5600
-Wire Wire Line
-	8850 5550 8850 5600
-Wire Wire Line
-	8850 5600 8700 5600
-Connection ~ 8700 5600
-Wire Wire Line
-	8700 5250 8700 5200
-Connection ~ 8700 5250
-Wire Wire Line
-	8700 5250 8850 5250
-$Comp
-L Device:C C31
-U 1 1 5F6DC4AB
-P 9550 5700
-F 0 "C31" H 9665 5746 50  0000 L CNN
-F 1 "0.1uF" H 9665 5655 50  0000 L CNN
-F 2 "Capacitor_SMD:C_0805_2012Metric" H 9588 5550 50  0001 C CNN
-F 3 "~" H 9550 5700 50  0001 C CNN
-F 4 "311-1140-1-ND" H 9550 5700 50  0001 C CNN "Digikey Part Number"
-F 5 "Yageo" H 9550 5700 50  0001 C CNN "Manufacturer_Name"
-F 6 "CC0805KRX7R9BB104" H 9550 5700 50  0001 C CNN "Manufacturer_Part_Number"
-F 7 "https://www.digikey.com.au/product-detail/en/yageo/CC0805KRX7R9BB104/311-1140-1-ND/303050" H 9550 5700 50  0001 C CNN "URL"
-F 8 "CC0805KRX7R9BB104" H 9550 5700 50  0001 C CNN "Part #"
-	1    9550 5700
-	1    0    0    -1
-$EndComp
-$Comp
-L Device:R R67
-U 1 1 5F6DC4B5
-P 9250 5950
-F 0 "R67" V 9450 5950 50  0000 C CNN
-F 1 "22K" V 9350 5950 50  0000 C CNN
-F 2 "Resistor_SMD:R_0805_2012Metric" V 9180 5950 50  0001 C CNN
-F 3 "~" H 9250 5950 50  0001 C CNN
-F 4 "YAG3773CT-ND" H 9250 5950 50  0001 C CNN "Digikey Part Number"
-F 5 "Yageo" H 9250 5950 50  0001 C CNN "Manufacturer_Name"
-F 6 "AC0805JR-0722KL" H 9250 5950 50  0001 C CNN "Manufacturer_Part_Number"
-F 7 "https://www.digikey.com.au/product-detail/en/yageo/AC0805JR-0722KL/YAG3773CT-ND/6006622" H 9250 5950 50  0001 C CNN "URL"
-	1    9250 5950
-	0    -1   -1   0
-$EndComp
-$Comp
-L Misc:KP234 U11
-U 1 1 5F6DC4BF
-P 8700 5950
-F 0 "U11" H 8271 6041 50  0000 R CNN
-F 1 "KP234" H 8271 5950 50  0000 R CNN
-F 2 "Misc:KP234" H 8271 5859 50  0000 R CNN
-F 3 "" H 8700 6550 50  0001 C CNN
-F 4 "448-KP234XTMA1CT-ND" H 8700 5950 50  0001 C CNN "Digikey Part Number"
-F 5 "Infineon" H 8700 5950 50  0001 C CNN "Manufacturer_Name"
-F 6 "KP234XTMA1" H 8700 5950 50  0001 C CNN "Manufacturer_Part_Number"
-F 7 "https://www.digikey.com.au/product-detail/en/infineon-technologies/KP234XTMA1/448-KP234XTMA1CT-ND/12718428" H 8700 5950 50  0001 C CNN "URL"
-	1    8700 5950
-	1    0    0    -1
-$EndComp
-Wire Wire Line
-	9550 5450 9550 5550
-Wire Wire Line
-	9400 5950 9550 5950
-Connection ~ 9550 5950
-Wire Wire Line
-	8450 6250 8500 6250
-Wire Wire Line
-	8500 6250 8700 6250
-Connection ~ 8500 6250
 $EndSCHEMATC
