File: PNPs/Miata NA6/Prior versions/v1.2/proto.sch (KiCad schematic (older format))
At the start: 11 parts, among them J3 Conn_01x06, J4 Conn_01x06, J5 Conn_01x06, J7 Conn_01x06

Commit message: NA6 PNP v1.3 files
Parts:
- R64: Digikey Part Number 311-1.00KCRCT-ND -> (none); Manufacturer_Name Yageo -> (none); Manufacturer_Part_Number RC0805FR-071KL -> (none); URL https://www.digikey.com/product-detail/en/yageo/RC0805FR-07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 -> (none)
Changed lines of the file:
@@
 F 2 "Resistor_SMD:R_0805_2012Metric_Pad1.15x1.40mm_HandSolder" V 6030 5400 50  0001 C CNN
 F 3 "~" H 6100 5400 50  0001 C CNN
-F 4 "Yageo" H -150 2350 50  0001 C CNN "Manufacturer_Name"
-F 5 "RC0805FR-071KL" H -150 2350 50  0001 C CNN "Manufacturer_Part_Number"
-F 6 "https://www.digikey.com/product-detail/en/yageo/RC0805FR-071KL/311-1.00KCRCT-ND/730391" H -150 2350 50  0001 C CNN "URL"
-F 7 "311-1.00KCRCT-ND" H -150 2350 50  0001 C CNN "Digikey Part Number"
+F 4 "" H -150 2350 50  0001 C CNN "Manufacturer_Name"
+F 5 "" H -150 2350 50  0001 C CNN "Manufacturer_Part_Number"
+F 6 "" H -150 2350 50  0001 C CNN "URL"
+F 7 "" H -150 2350 50  0001 C CNN "Digikey Part Number"
 	1    6100 5400
 	1    0    0    -1
